File: Any-Screen-Touch-Screen_AnchorMod/Any-Screen-Touch-Screen_AnchorMod.kicad_sch (KiCad schematic)
At the start: 28 parts, among them P1 USB_C_Plug_USB2.0, Q2 S8050, Q3 S8050, SW1 SW_Push, SW2 SW_Push, U1 ESP32-S3-WROOM-1, U2 CP2104

Commit message: Merged power subsystem into pen and anchor schematics, changed input/output devices to pin connectors; also updated lab notebook
Parts:
- removed D1, D2, D3, D4: LED, symbol Device:LED
- removed SW1, SW2: SW_Push, symbol Switch:SW_Push
- added C5: 1 μF, Capacitor_SMD:C_0805_2012Metric_Pad1.18x1.45mm_HandSolder, symbol Device:C
- added C6, C7: 10 μF, Capacitor_SMD:C_0805_2012Metric_Pad1.18x1.45mm_HandSolder, symbol Device:C
- added C8: 0.47 μF, symbol Device:C
- added D5: 1N5819, Diode_THT:D_DO-41_SOD81_P10.16mm_Horizontal, symbol Diode:1N5819
- added H1, H2, H3, H4: MountingHole, symbol Mechanical:MountingHole
- added J1: Reset button, symbol Connector_Generic:Conn_01x02
- added J2: Flash button, symbol Connector_Generic:Conn_01x02
- added J3: Power Switch, symbol Connector_Generic:Conn_01x02
- added J4: Battery Terminals, symbol Connector_Generic:Conn_01x02
- added J5: LED1, symbol Connector_Generic:Conn_01x02
- added J6: LED2, symbol Connector_Generic:Conn_01x02
- added J7: LED3, symbol Connector_Generic:Conn_01x02
- added J8: LED4, symbol Connector_Generic:Conn_01x02
- added L1: 4.7 μH, symbol Device:L
- added Q1: IRLZ44N, Package_TO_SOT_THT:TO-220-3_Vertical, symbol Transistor_FET:IRLZ44N
- added R13, R14, R15: 10kΩ, symbol Device:R
- added U3: BQ27441-G1, Package_SON:Texas_S-PDSO-N12, symbol Battery_Management:BQ27441-G1
- added U4: TLV62569DBV, Package_TO_SOT_SMD:SOT-23-5, symbol Regulator_Switching:TLV62569DBV
- C1, C2, C3, C4: footprint (none) -> Capacitor_SMD:C_0805_2012Metric_Pad1.18x1.45mm_HandSolder
Connections:
- net +3.3V: now also C7.1, L1.2
- net GND: now also C5.2, C7.2, C8.2, D5.2 (A), J1.2 (Pin_2), J4.2 (Pin_2), J5.2 (Pin_2), J6.2 (Pin_2), J7.2 (Pin_2), J8.2 (Pin_2), U3.3 (V_{SS})
- net RESET_ESP: now also J1.1 (Pin_1)
- net USB_VBUS: no longer P1.A4 (VBUS), P1.A9 (VBUS), P1.B4 (VBUS), P1.B9 (VBUS)
- net at R7.1: now also J7.1 (Pin_1)
- net MCU GPIO: now reaches U1.23 (IO21)
- net MCU GPIO: now also R15.2, U3.12 (GPOUT)
- net I2C Clock: now reaches U1.38 (IO2)
- net I2C Clock: now also R13.2, U3.2 (SCL)
- net I2C Data: now reaches U1.39 (IO1)
- net I2C Data: now also R14.2, U3.1 (SDA)
- net at R5.1: now also J5.1 (Pin_1)
- net at R9.2: now also J2.1 (Pin_1)
- net at R8.1: now also J8.1 (Pin_1)
- net at R6.1: now also J6.1 (Pin_1)
- new net: C6.1, Q1.2 (D)
- new net: D5.1 (K), L1.1, Q1.3 (S)
- new net: C8.1, U3.5 (V_{DD})
- new net: C5.1, C6.2, J3.2 (Pin_2), R13.1, R14.1, R15.1, U3.6 (BAT)
- new net: J3.1 (Pin_1), J4.1 (Pin_1)
- new net: P1.A4 (VBUS), P1.A9 (VBUS), P1.B4 (VBUS), P1.B9 (VBUS)
- new net MCU PWM: Q1.1 (G)
Other:
- note added: "3.3V Buck Converter"
- note added: "Battery Fuel Gauge"
- note added: "Microcontroller"
- note added: "USB-to-UART"
- moved on the sheet: C1, C2, C3, C4, DWM1, P1, Q2, Q3, R1, R10, R11, R12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

Commit message: Started PCB layout and organized components
Parts:
- removed D5: 1N5819, Diode_THT:D_DO-41_SOD81_P10.16mm_Horizontal, symbol Diode:1N5819
- removed Q1: IRLZ44N, Package_TO_SOT_THT:TO-220-3_Vertical, symbol Transistor_FET:IRLZ44N
- removed Q2, Q3: S8050, Package_TO_SOT_THT:TO-92_Inline, symbol Transistor_BJT:S8050
- removed R11, R12: 1k, symbol Device:R
- removed U4: TLV62569DBV, Package_TO_SOT_SMD:SOT-23-5, symbol Regulator_Switching:TLV62569DBV
- added U5: TPS63001, Package_SON:Texas_DRC0010J_ThermalVias, symbol Regulator_Switching:TPS63001
- C7: value 10 μF -> 33 μF
- C8: footprint (none) -> Capacitor_SMD:C_0805_2012Metric_Pad1.18x1.45mm_HandSolder
- H1, H2, H3, H4: footprint (none) -> MountingHole:MountingHole_3.2mm_M3
- J1, J2, J3, J4, J5, J6, J7, J8: footprint (none) -> Connector_Molex:Molex_KK-254_AE-6410-02A_1x02_P2.54mm_Vertical
- L1: value 4.7 μH -> 2.2μH; footprint (none) -> footprints:IND_MSS5131_COC
- P1: footprint (none) -> Connector_USB:USB_C_Plug_Molex_105444
- R1, R10, R13, R14, R15, R2, R3, R4, R5, R6, R7, R8, R9: footprint (none) -> Resistor_SMD:R_0805_2012Metric_Pad1.20x1.40mm_HandSolder
- U2: footprint Package_DFN_QFN:QFN-24-1EP_4x4mm_P0.5mm_EP2.6x2.6mm -> Package_DFN_QFN:QFN-24-1EP_4x4mm_P0.5mm_EP2.7x2.7mm_ThermalVias
Connections:
- net +3.3V: now also U5.1 (VOUT), U5.10 (FB); no longer L1.2
- net GND: now also C6.1, U5.11 (PGND), U5.3 (PGND), U5.9 (GND)
- net at L1.1: now also U5.2 (L2)
- net at C5.1, C6.2, J3.2 (Pin_2)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: now also U5.5 (VIN), U5.6 (EN), U5.7 (PS/SYNC), U5.8 (VINA)
- new net: L1.2, U5.4 (L1)
Other:
- moved on the sheet: C6
