File: Any-Screen-Touch-Screen_Pen/Any-Screen-Touch-Screen_Pen.kicad_sch (KiCad schematic)
At the start: 33 parts, among them J1 PEN_BUTTON, P1 USB_C_Plug_USB2.0, Q1 S8050, Q2 S8050, SW1 SW_Push, SW2 SW_Push, U1 CP2104, U2 ESP32-S3-WROOM-1, U4 LSM6DSL

Commit message: Merged power subsystem into pen and anchor schematics, changed input/output devices to pin connectors; also updated lab notebook
Parts:
- removed D1, D2, D3, D4: LED, symbol Device:LED
- removed SW1, SW2: SW_Push, symbol Switch:SW_Push
- added C10: 0.47 μF, symbol Device:C
- added C7: 1 μF, symbol Device:C
- added C8, C9: 10 μF, symbol Device:C
- added D5: 1N5819, Diode_THT:D_DO-41_SOD81_P10.16mm_Horizontal, symbol Diode:1N5819
- added H1, H2, H3, H4: MountingHole, symbol Mechanical:MountingHole
- added J2: Reset button, symbol Connector_Generic:Conn_01x02
- added J3: Flash button, symbol Connector_Generic:Conn_01x02
- added J4: Battery Terminals, symbol Connector_Generic:Conn_01x02
- added J5: Power Switch, symbol Connector_Generic:Conn_01x02
- added J6: LED1, symbol Connector_Generic:Conn_01x02
- added J7: LED2, symbol Connector_Generic:Conn_01x02
- added J8: LED3, symbol Connector_Generic:Conn_01x02
- added J9: LED4, symbol Connector_Generic:Conn_01x02
- added L1: 4.7 μH, symbol Device:L
- added Q3: IRLZ44N, Package_TO_SOT_THT:TO-220-3_Vertical, symbol Transistor_FET:IRLZ44N
- added R14, R15, R16: 10kΩ, symbol Device:R
- added U3: BQ27441-G1, Package_SON:Texas_S-PDSO-N12, symbol Battery_Management:BQ27441-G1
- added U5: AMS1117-1.8, Package_TO_SOT_SMD:SOT-223-3_TabPin2, symbol Regulator_Linear:AMS1117-1.8
Connections:
- net +3.3V: now also C9.1, L1.2, U5.3 (VI)
- net GND: now also C10.2, C7.2, C9.2, D5.2 (A), J2.1 (Pin_1), J3.1 (Pin_1), J4.1 (Pin_1), J6.2 (Pin_2), J7.2 (Pin_2), J8.2 (Pin_2), J9.2 (Pin_2), U3.3 (V_{SS}), U5.1 (GND)
- net RESET_ESP: now also J2.2 (Pin_2)
- net USB_VBUS: no longer P1.A4 (VBUS), P1.A9 (VBUS), P1.B4 (VBUS), P1.B9 (VBUS)
- net at R11.1: now also J8.1 (Pin_1)
- net at R4.2: now also J3.2 (Pin_2)
- net at R9.1: now also J6.1 (Pin_1)
- net at R12.1: now also J9.1 (Pin_1)
- net at R10.1: now also J7.1 (Pin_1)
- net MCU GPIO: now reaches U2.10 (IO17)
- net MCU GPIO: now also R16.2, U3.12 (GPOUT)
- net I2C Data: now reaches U2.8 (IO15)
- net I2C Data: now also R15.2, U3.1 (SDA)
- net I2C Clock: now reaches U2.9 (IO16)
- net I2C Clock: now also R14.2, U3.2 (SCL)
- net Vout - 1.8V renamed +1.8V
- net +1.8V: now also U5.2 (VO)
- new net: C8.1, Q3.2 (D)
- new net: D5.1 (K), L1.1, Q3.3 (S)
- new net: J4.2 (Pin_2), J5.1 (Pin_1)
- new net: C7.1, C8.2, J5.2 (Pin_2), R14.1, R15.1, R16.1, U3.6 (BAT)
- new net: C10.1, U3.5 (V_{DD})
- new net: P1.A4 (VBUS), P1.A9 (VBUS), P1.B4 (VBUS), P1.B9 (VBUS)
- new net MCU PWM: Q3.1 (G)
Other:
- note added: "1.8V LDO"
- note added: "3.3V Buck Converter"
- note added: "Battery Fuel Gauge"
- note removed: "1"

Commit message: Started PCB layout and organized components
Parts:
- removed D5: 1N5819, Diode_THT:D_DO-41_SOD81_P10.16mm_Horizontal, symbol Diode:1N5819
- removed Q3: IRLZ44N, Package_TO_SOT_THT:TO-220-3_Vertical, symbol Transistor_FET:IRLZ44N
- added C11: 22 μF, Capacitor_SMD:C_0805_2012Metric_Pad1.18x1.45mm_HandSolder, symbol Device:C
- added U6: TPS63001, Package_SON:Texas_DRC0010J_ThermalVias, symbol Regulator_Switching:TPS63001
- C8: footprint (none) -> Capacitor_SMD:C_0805_2012Metric_Pad1.18x1.45mm_HandSolder
- C9: value 10 μF -> 33 μF; footprint (none) -> Capacitor_SMD:C_0805_2012Metric_Pad1.18x1.45mm_HandSolder
- L1: value 4.7 μH -> 2.2μF
Connections:
- net +1.8V: now also C11.1
- net +3.3V: now also U6.1 (VOUT), U6.10 (FB); no longer L1.2
- net GND: now also C8.1, J4.2 (Pin_2), C11.2, U6.11 (PGND), U6.3 (PGND), U6.9 (GND); no longer J4.1 (Pin_1)
- net at L1.1: now also U6.2 (L2)
- net at J5.1 (Pin_1): now also J4.1 (Pin_1); no longer J4.2 (Pin_2)
- net at C7.1, C8.2, J5.2 (Pin_2)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: now also U6.5 (VIN), U6.6 (EN), U6.7 (PS/SYNC), U6.8 (VINA)
- new net: L1.2, U6.4 (L1)
Other:
- moved on the sheet: U5
